File: cwkeyer/cwkeyer.kicad_pcb (KiCad board)
At the start: 2 copper layers, 18 x 15.5 mm, 8 parts, among them J1 Conn_01x05, J2 Conn_01x03, Q1 S8050, U1 ATtiny85-20SU

Commit message: Re-route the PCB.
Connections:
- J1 pad 1: SW -> PAD_L
- J1 pad 2: PAD_L -> PAD_R
- J1 pad 3: PAD_R -> KEY
- J1 pad 4: TONE -> SW
- J1 pad 5: KEY -> TONE
Routing:
- net SW: track 24.4 -> 13.0 mm
- net KEY: track 12.1 -> 5.77 mm
- net GND: track 0.00 -> 1.86 mm, vias 6 -> 4
- net PAD_L: track 13.3 -> 14.7 mm
- net TONE: track 12.6 -> 13.9 mm, vias 1 -> 0
- net PAD_R: track 12.6 -> 13.2 mm, vias 2 -> 0
